File: HorizonPC.kicad_pcb (KiCad board)
At the start: 8 copper layers, 50 x 50 mm, 256 parts, among them J2 MSD-1-A, J3 Conn_01x05_Pin, J4 DF40C-90DP-0.4V(51), SW1 219-5LPSTR, U1 R9A07G043F05GBG#BC0, U11 TPS552892RYQR, U12 TPS2051CDBV, U13 USBLC6-2SC6, U14 DDR4, U15 DDR4, U2 TPS51200DRC, U3 S25FL256SAGNFI011, U4 DA9062-52AM1, U5 ATA6561-GBQW-N, U6 ATA6561-GBQW-N, U7 SM662GXC, Y1 32.768KHz, Y2 DSC6101JE3B-24MHz

Commit message: Update
Parts:
- removed C193, C195, C206, C84, C86: 47n, Capacitor_SMD:C_0402_1005Metric
- added C147: 100n, Capacitor_SMD:C_0402_1005Metric, B.Cu at (187.3, 69.3)
- added C148: 100n, Capacitor_SMD:C_0402_1005Metric, B.Cu at (188.3, 69.3)
- added C149: 100n, Capacitor_SMD:C_0402_1005Metric, B.Cu at (179.5, 69.3)
- added C152: 100n, Capacitor_SMD:C_0402_1005Metric, B.Cu at (182.1, 69.3)
- added C153: 100n, Capacitor_SMD:C_0402_1005Metric, B.Cu at (177.9, 69.3)
- added C154: 100n, Capacitor_SMD:C_0402_1005Metric, B.Cu at (189.9, 69.3)
- added C156: 100n, Capacitor_SMD:C_0402_1005Metric, B.Cu at (184.7, 69.3)
- added C157: 100n, Capacitor_SMD:C_0402_1005Metric, B.Cu at (185.7, 69.3)
- added C158: 100n, Capacitor_SMD:C_0402_1005Metric, B.Cu at (180.5, 69.3)
- added C159: 100n, Capacitor_SMD:C_0402_1005Metric, B.Cu at (183.1, 69.3)
- added C167: 100n, Capacitor_SMD:C_0402_1005Metric, B.Cu at (195.1, 69.3)
- added C168: 100n, Capacitor_SMD:C_0402_1005Metric, B.Cu at (193.5, 69.3)
- added C169: 100n, Capacitor_SMD:C_0402_1005Metric, B.Cu at (192.5, 69.3)
- added C170: 100n, Capacitor_SMD:C_0402_1005Metric, B.Cu at (190.9, 69.3)
- added D3: 12V, Diode_SMD:D_SOD-123, F.Cu at (217.4, 112.5)
- added F1: 8A, Fuse:Fuse_0603_1608Metric, F.Cu at (222.3, 112.1)
- added Q1: PMOS, Package_SO:PowerPAK_SO-8_Single, F.Cu at (219.0, 107.5)
- added R94: 47k, Resistor_SMD:R_0402_1005Metric, F.Cu at (221.7, 114.3)
- C192, C194: value 47n -> 100n
- R38: moved to B.Cu
- moved R38 72.3 mm to (185.2, 76.7), turned to 90 degrees
- moved R3 57.7 mm to (165.2, 101.0), turned to -90 degrees
- moved R4 56.7 mm to (164.2, 101.0), turned to -90 degrees
- moved R5 55.8 mm to (163.2, 101.0), turned to -90 degrees
- moved RN7 26.8 mm to (194.3, 69.4), turned to 90 degrees
- moved RN6 23.0 mm to (191.7, 69.4), turned to 90 degrees
- moved RN5 19.2 mm to (189.1, 69.4), turned to 90 degrees
- moved RN4 15.5 mm to (186.5, 69.4), turned to 90 degrees
- moved RN3 11.7 mm to (183.9, 69.4), turned to 90 degrees
- moved RN2 7.91 mm to (181.3, 69.4), turned to 90 degrees
- moved RN1 4.17 mm to (178.7, 69.4), turned to 90 degrees
- moved R39 3.39 mm to (178.1, 93.4)
- moved C219 2.47 mm to (174.8, 76.5)
- moved C38 2.24 mm to (208.0, 77.0)
- moved C39 2.24 mm to (209.5, 70.8)
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Connections:
- RN1 pad 1: DDR_BA0 -> DDR_A13
- RN1 pad 2: DDR_BG0 -> DDR_A11
- RN1 pad 3: DDR_WE -> DDR_A7
- RN1 pad 4: DDR_CKE -> DDR_A9
- RN2 pad 1: DDR_A8 -> DDR_A2
- RN2 pad 2: DDR_A6 -> DDR_A5
- RN2 pad 3: DDR_ODT0 -> DDR_A1
- RN2 pad 4: DDR_A4 -> DDR_A6
- RN3 pad 1: DDR_A0 -> DDR_BA0
- RN3 pad 2: unconnected-(RN3-R2.1-Pad2) -> DDR_BA1
- RN3 pad 3: unconnected-(RN3-R3.1-Pad3) -> DDR_A8
- RN3 pad 4: DDR_A11 -> DDR_A3
- RN4 pad 1: DDR_ACT -> DDR_A0
- RN4 pad 2: DDR_ODT1 -> DDR_CAS
- RN4 pad 4: DDR_A2 -> DDR_A4
- RN5 pad 1: DDR_CAS -> DDR_CS0
- RN5 pad 2: DDR_A12 -> DDR_CS1
- RN5 pad 3: DDR_RAS -> DDR_ODT0
- RN5 pad 4: DDR_CS1 -> DDR_A12
- RN6 pad 1: DDR_A5 -> DDR_RAS
- RN6 pad 2: DDR_A1 -> DDR_BG0
- RN6 pad 3: DDR_BA1 -> DDR_ACT
- RN6 pad 4: DDR_A3 -> DDR_ODT1
- RN7 pad 1: DDR_CS0 -> DDR_WE
- RN7 pad 2: DDR_A13 -> DDR_CKE
- RN7 pad 3: DDR_A7 -> unconnected-(RN7-R3.1-Pad3)
- RN7 pad 4: DDR_A9 -> unconnected-(RN7-R4.1-Pad4)
- U1 pad A24: DDR_A13 -> DDR_A11
- U1 pad AA24: DDR_DQ10 -> DDR_DQ14
- U1 pad AC24: DDR_DQ15 -> DDR_DQ10
- U1 pad AD23: DDR_DQ9 -> DDR_DQ8
- U1 pad AD24: DDR_DQ8 -> DDR_DQ11
- U1 pad AE24: DDR_DQ11 -> DDR_DQ9
- U1 pad B25: DDR_A11 -> DDR_A13
- U1 pad C24: DDR_A2 -> DDR_A1
- U1 pad D23: DDR_A8 -> DDR_A3
- U1 pad D25: DDR_A1 -> DDR_A5
- U1 pad E24: DDR_BA0 -> DDR_A2
- U1 pad E25: DDR_A5 -> DDR_BA1
- U1 pad F23: DDR_BA1 -> DDR_A10
- U1 pad F25: DDR_A6 -> DDR_CAS
- U1 pad G25: DDR_A10 -> DDR_A12
- U1 pad H23: DDR_A12 -> DDR_A8
- U1 pad H24: DDR_A0 -> DDR_A6
- U1 pad H25: DDR_A4 -> DDR_A0
- U1 pad J24: DDR_A3 -> DDR_A4
- U1 pad J25: DDR_CS0 -> DDR_BA0
- U1 pad K23: DDR_CAS -> DDR_WE
- U1 pad K25: DDR_BG0 -> DDR_RAS
- U1 pad L23: DDR_CS1 -> DDR_ODT0
- U1 pad L24: DDR_ACT -> DDR_CS0
- U1 pad L25: DDR_RAS -> DDR_ACT
- U1 pad M24: DDR_ODT0 -> DDR_CS1
- U1 pad N23: DDR_ODT1 -> DDR_BG0
- U1 pad N24: DDR_WE -> DDR_ODT1
- U1 pad T23: DDR_DQ3 -> DDR_DQ2
- U1 pad T24: DDR_DQ5 -> DDR_DQ4
- U1 pad T25: DDR_DQ2 -> DDR_DQ5
- U1 pad U25: DDR_DQ4 -> DDR_DQ3
- U1 pad W23: DDR_DQ14 -> DDR_DQ15
- U1 pad W24: DDR_DQ1 -> DDR_DQ0
- U1 pad Y25: DDR_DQ0 -> DDR_DQ1
Routing:
- net GND: track 156.2 -> 131.6 mm, vias 252 -> 372
- net +1.2V: track 119.7 -> 100.2 mm, vias 41 -> 43
- net VTT_REF: track 35.5 -> 17.3 mm, vias 4 -> 3
- net SD1_D3: track 18.0 -> 34.4 mm, vias 1 -> 2
- net SD1_D2: track 18.7 -> 34.0 mm, vias 1 -> 2
- net SD1_D1: track 10.6 -> 25.3 mm, vias 1 -> 2
- net SD1_CMD: track 16.2 -> 30.7 mm, vias 1 -> 2
- net SD1_D0: track 12.8 -> 25.5 mm, vias 1 -> 2
- net SD1_CLK: track 16.0 -> 27.0 mm
- net VTT: track 41.0 -> 51.3 mm, vias 0 -> 17
- net DDR_CS0: track 27.8 -> 37.3 mm
- net SD1_DET: track 10.3 -> 16.6 mm, vias 2 -> 3
- net DDR_RAS: track 37.7 -> 43.0 mm
- net DDR_CS1: track 37.1 -> 32.1 mm, vias 2 -> 3
- net DDR_CK-: track 23.9 -> 28.6 mm, vias 3 -> 4
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- added copper zone on B.Cu, net GND
- added copper zone on F.Cu, net GND
- added copper zone on In2.Cu, net GND
- added copper zone on In5.Cu, net GND
- added copper zone on F.Cu, net VTT
Other:
- board size 50 x 50 mm -> 52 x 52 mm

Commit message: Update
Parts:
- removed U13: USBLC6-2SC6, Package_TO_SOT_SMD:SOT-23-6
- added C140: 100n, Capacitor_SMD:C_0402_1005Metric, B.Cu at (190.9, 103.0)
- added C141: 100n, Capacitor_SMD:C_0402_1005Metric, B.Cu at (184.0, 101.9)
- added C226: 100n, Capacitor_SMD:C_0402_1005Metric, F.Cu at (174.8, 82.5)
- added C44: 100n, Capacitor_SMD:C_0402_1005Metric, F.Cu at (177.5, 110.0)
- added D4: CDSOD323-T05S, Diode_SMD:D_SOD-323, F.Cu at (202.3, 82.0)
- added D5: CDSOD323-T03S, Diode_SMD:D_SOD-323, F.Cu at (172.8, 100.3)
- added D6: CDSOD323-T05S, Diode_SMD:D_SOD-323, F.Cu at (196.1, 94.7)
- added J5: BK13H-30DP/2-0.35V05(895), HorizonPC:BK13H-30DP_2-0.35V05, B.Cu at (177.1, 91.0)
- added J6: BK13H-30DP/2-0.35V05(895), HorizonPC:BK13H-30DP_2-0.35V05, B.Cu at (197.2, 92.0)
- added U10: ECMF02-2AMX6, Package_DFN_QFN:ST_UQFN-6L_1.5x1.7mm_P0.5mm, B.Cu at (204.4, 100.2)
- added U8: PUSB3TB6AZ, HorizonPC:XSON7_PUSB3_NEX, B.Cu at (176.7, 105.9)
- added U9: ECMF02-2AMX6, Package_DFN_QFN:ST_UQFN-6L_1.5x1.7mm_P0.5mm, B.Cu at (204.4, 103.1)
- R89, R90, R91, R92: moved to B.Cu
- TP1: footprint TestPoint:TestPoint_Pad_D2.0mm -> TestPoint:TestPoint_Pad_D1.0mm
- moved R6 99.0 mm to (206.2, 99.5), turned to -90 degrees
- moved R2 98.8 mm to (206.2, 101.3), turned to 90 degrees
- moved TP1 70.6 mm to (161.7, 99.5)
- moved J3 69.4 mm to (209.9, 110.5), turned to 180 degrees
- moved R7 57.9 mm to (164.9, 101.0), turned to -90 degrees
- moved R94 32.7 mm to (203.8, 86.9), turned to 90 degrees
- moved R78 28.3 mm to (152.8, 110.1)
- moved R79 28.3 mm to (152.8, 112.0)
- moved Q1 26.4 mm to (198.6, 90.8), turned to 180 degrees
- moved F1 25.9 mm to (203.2, 94.7), turned to -90 degrees
- moved D3 25.8 mm to (203.8, 90.5), turned to 90 degrees
- moved R92 24.2 mm to (180.9, 105.6), turned to 90 degrees
- moved R91 22.2 mm to (179.0, 105.9), turned to 90 degrees
- moved R89 20.4 mm to (178.7, 103.5)
- moved R90 19.8 mm to (178.8, 104.5)
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Connections:
- C160 pad 1: GND -> +3.3V
- C160 pad 2: +3.3V -> GND
- J3 pad 3: JTAG_TDO -> JTAG_TRST#
- J3 pad 4: JTAG_TDI -> JTAG_TDO
- J3 pad 5: JTAG_TRST# -> JTAG_TDI
- J4 pad 10a: unconnected-(J4-Pin_10a-Pad10a) -> ETH_MDIO
- J4 pad 10b: unconnected-(J4-Pin_10b-Pad10b) -> MTU1_A
- J4 pad 11a: unconnected-(J4-Pin_11a-Pad11a) -> GND
- J4 pad 11b: unconnected-(J4-Pin_11b-Pad11b) -> GND
- J4 pad 12a: unconnected-(J4-Pin_12a-Pad12a) -> ETH_RXD3
- J4 pad 12b: unconnected-(J4-Pin_12b-Pad12b) -> ETH_TXD3
- J4 pad 13a: unconnected-(J4-Pin_13a-Pad13a) -> ETH_RXD2
- J4 pad 13b: unconnected-(J4-Pin_13b-Pad13b) -> ETH_TXD2
- J4 pad 14a: unconnected-(J4-Pin_14a-Pad14a) -> GND
- J4 pad 14b: unconnected-(J4-Pin_14b-Pad14b) -> GND
- J4 pad 15a: unconnected-(J4-Pin_15a-Pad15a) -> ETH_RXD1
- J4 pad 15b: unconnected-(J4-Pin_15b-Pad15b) -> ETH_TXD1
- J4 pad 16a: unconnected-(J4-Pin_16a-Pad16a) -> ETH_RXD0
- J4 pad 16b: unconnected-(J4-Pin_16b-Pad16b) -> ETH_TXD0
- J4 pad 17a: unconnected-(J4-Pin_17a-Pad17a) -> GND
- J4 pad 17b: unconnected-(J4-Pin_17b-Pad17b) -> GND
- J4 pad 18a: unconnected-(J4-Pin_18a-Pad18a) -> ETH_RXC
- J4 pad 18b: unconnected-(J4-Pin_18b-Pad18b) -> ETH_TXC
- J4 pad 19a: unconnected-(J4-Pin_19a-Pad19a) -> GND
- J4 pad 19b: unconnected-(J4-Pin_19b-Pad19b) -> GND
- J4 pad 1a: unconnected-(J4-Pin_1a-Pad1a) -> USB_ESD+
- J4 pad 1b: unconnected-(J4-Pin_1b-Pad1b) -> JTAG_TDI
- J4 pad 20a: unconnected-(J4-Pin_20a-Pad20a) -> ETH_RX_CTL
- J4 pad 20b: unconnected-(J4-Pin_20b-Pad20b) -> ETH_TX_CTL
- J4 pad 21a: unconnected-(J4-Pin_21a-Pad21a) -> GND
- J4 pad 21b: unconnected-(J4-Pin_21b-Pad21b) -> GND
- J4 pad 22a: unconnected-(J4-Pin_22a-Pad22a) -> CSI_D3+
- J4 pad 23a: unconnected-(J4-Pin_23a-Pad23a) -> CSI_D3-
- J4 pad 24a: unconnected-(J4-Pin_24a-Pad24a) -> GND
- J4 pad 25a: unconnected-(J4-Pin_25a-Pad25a) -> CSI_D1-
- J4 pad 26a: unconnected-(J4-Pin_26a-Pad26a) -> CSI_D1+
- J4 pad 27a: unconnected-(J4-Pin_27a-Pad27a) -> GND
- J4 pad 28a: unconnected-(J4-Pin_28a-Pad28a) -> CSI_CLK-
- J4 pad 29a: unconnected-(J4-Pin_29a-Pad29a) -> CSI_CLK+
- J4 pad 2a: unconnected-(J4-Pin_2a-Pad2a) -> USB_ESD-
- J4 pad 2b: unconnected-(J4-Pin_2b-Pad2b) -> JTAG_TDO
- J4 pad 30a: unconnected-(J4-Pin_30a-Pad30a) -> GND
- J4 pad 31a: unconnected-(J4-Pin_31a-Pad31a) -> CSI_D0-
- J4 pad 32a: unconnected-(J4-Pin_32a-Pad32a) -> CSI_D0+
- J4 pad 33a: unconnected-(J4-Pin_33a-Pad33a) -> GND
- J4 pad 34a: unconnected-(J4-Pin_34a-Pad34a) -> CSI_D2-
- J4 pad 35a: unconnected-(J4-Pin_35a-Pad35a) -> CSI_D2+
- J4 pad 36a: unconnected-(J4-Pin_36a-Pad36a) -> GND
- J4 pad 37a: unconnected-(J4-Pin_37a-Pad37a) -> GPIO0_33
- J4 pad 38a: unconnected-(J4-Pin_38a-Pad38a) -> GND
- J4 pad 39a: unconnected-(J4-Pin_39a-Pad39a) -> SPI2_MISO
- J4 pad 3a: unconnected-(J4-Pin_3a-Pad3a) -> USB_MAIN_ESD-
- J4 pad 3b: unconnected-(J4-Pin_3b-Pad3b) -> JTAG_TRST#
- J4 pad 40a: unconnected-(J4-Pin_40a-Pad40a) -> SPI2_SSL
- J4 pad 41a: unconnected-(J4-Pin_41a-Pad41a) -> SPI2_CLK
- J4 pad 42a: unconnected-(J4-Pin_42a-Pad42a) -> SPI2_MOSI
- J4 pad 43a: unconnected-(J4-Pin_43a-Pad43a) -> GND
- J4 pad 43b: unconnected-(J4-Pin_43b-Pad43b) -> GND
- J4 pad 4a: unconnected-(J4-Pin_4a-Pad4a) -> USB_MAIN_ESD+
- J4 pad 4b: unconnected-(J4-Pin_4b-Pad4b) -> JTAG_TCK
- J4 pad 5a: unconnected-(J4-Pin_5a-Pad5a) -> GND
- J4 pad 5b: unconnected-(J4-Pin_5b-Pad5b) -> JTAG_TMS
- J4 pad 6a: unconnected-(J4-Pin_6a-Pad6a) -> PWR_ONKEY
- J4 pad 6b: unconnected-(J4-Pin_6b-Pad6b) -> NMI
- J4 pad 7a: unconnected-(J4-Pin_7a-Pad7a) -> SYS_EN
- J4 pad 7b: unconnected-(J4-Pin_7b-Pad7b) -> MTU1_D
- J4 pad 8a: unconnected-(J4-Pin_8a-Pad8a) -> MAIN_RESET
- J4 pad 8b: unconnected-(J4-Pin_8b-Pad8b) -> MTU1_C
- J4 pad 9a: unconnected-(J4-Pin_9a-Pad9a) -> ETH_MDC
- J4 pad 9b: unconnected-(J4-Pin_9b-Pad9b) -> MTU1_B
- R18 pad 1: VSD1 -> +3.3V
- R2 pad 1: +5V_EXT -> +5V
- R6 pad 1: +5V_EXT -> +5V
- SW1 pad 6: VSD1 -> +3.3V
- SW1 pad 7: +1.8V -> +3.3V
- U1 pad A12: GPIO3_33 -> GPIO9_33
- U1 pad A14: LDO2_EN -> GPIO7_33
- U1 pad A17: CAN0_STBY -> GPIO2_33
- U1 pad A18: unconnected-(U1Power-NC-PadA18) -> ADC_CH1_ARM
- U1 pad A19: MAIN_SCL -> PWR_SCL
- U1 pad A20: MAIN_SDA -> PWR_SDA
- U1 pad A3: GPIO8_33 -> LDO3_EN
- U1 pad AC15: GPIO2_33 -> CAN0_STBY
- U1 pad AC16: GPIO1_33 -> CAN1_STBY
- U1 pad AD10: unconnected-(U1Power-NC-PadAD10) -> CSI_D1+
- U1 pad AD11: unconnected-(U1Power-NC-PadAD11) -> CSI_CLK+
- U1 pad AD12: unconnected-(U1Power-NC-PadAD12) -> CSI_D0+
- U1 pad AD13: ADC_CH1 -> CSI_D2+
- U1 pad AD9: unconnected-(U1Power-NC-PadAD9) -> CSI_D3+
- U1 pad AE10: unconnected-(U1Power-NC-PadAE10) -> CSI_D1-
- U1 pad AE11: unconnected-(U1Power-NC-PadAE11) -> CSI_CLK-
- U1 pad AE12: unconnected-(U1Power-NC-PadAE12) -> CSI_D0-
- U1 pad AE13: ADC_CH0 -> CSI_D2-
- U1 pad AE9: unconnected-(U1Power-NC-PadAE9) -> CSI_D3-
- U1 pad B12: PWR_WDT -> GPIO5_33
- U1 pad B14: LDO3_EN -> GPIO8_33
- U1 pad B17: CAN1_STBY -> GPIO1_33
- U1 pad B18: unconnected-(U1Power-NC-PadB18) -> ADC_CH0_ARM
- U1 pad B19: PWR_SCL -> MAIN_SCL
- U1 pad B2: GPIO5_33 -> PWR_WDT
- U1 pad B20: PWR_SDA -> MAIN_SDA
- U1 pad B3: GPIO9_33 -> LDO2_EN
- U1 pad B4: GPIO7_33 -> LDO4_EN
- U1 pad F16: LDO4_EN -> GPIO3_33
- U1 pad F17: unconnected-(U1Power-NC-PadF17) -> +1.8V
- U1 pad Y11: unconnected-(U1Power-NC-PadY11) -> +1.8V
- U1 pad Y12: unconnected-(U1Power-NC-PadY12) -> +1.8V
- U1 pad Y15: unconnected-(U1Power-NC-PadY15) -> +1.1V
Routing:
- net +3.3V: track 65.2 -> 190.7 mm, vias 35 -> 40
- net +1.8V: track 22.4 -> 136.2 mm, vias 21 -> 27
- net +1.2V: track 100.2 -> 212.9 mm, vias 43 -> 49
- net VPP: track 8.36 -> 108.9 mm, vias 5 -> 8
- net +5V: track 51.8 -> 131.1 mm, vias 17 -> 24
- net PWR_ONKEY: track 1.05 -> 71.5 mm, vias 1 -> 3
- net MAIN_RESET: track 1.90 -> 70.8 mm, vias 1 -> 3
- net CAN1_TXD: track 0.00 -> 62.8 mm, vias 0 -> 2
- net CAN1_RXD: track 1.15 -> 61.6 mm, vias 0 -> 2
- net VSD1: track 18.3 -> 77.8 mm, vias 6 -> 8
- net CAN0_TXD: track 0.55 -> 60.0 mm, vias 0 -> 2
- net CAN0_RXD: track 0.00 -> 58.3 mm, vias 0 -> 2
- net PWR_RESET: track 0.95 -> 46.3 mm, vias 0 -> 4
- net VETH: track 4.20 -> 46.1 mm, vias 2 -> 3
- net ETH_RX_CTL: track 0.35 -> 41.8 mm, vias 0 -> 2
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- added copper zone on In2.Cu, net +1.1V
- added copper zone on B.Cu, net +5V_USB
- added copper zone on F.Cu, net Net-(D3-K)
- added copper zone on B.Cu, net VMAIN_RAW
- added copper zone on F.Cu, net VMAIN_RAW
- added copper zone on F.Cu, net VPP
