File: HorizonPC.kicad_sch (KiCad schematic)
At the start: 269 parts, among them J2 MSD-1-A, J3 Conn_01x05_Pin, J4 DF40C-90DP-0.4V(51), Q1 PMOS, SW1 219-5LPSTR, U1 R9A07G043F05GBG#BC0, U11 TPS552892RYQR, U12 TPS2051CDBV, U13 USBLC6-2SC6, U14 DDR4, U15 DDR4, U2 TPS51200DRC, U3 S25FL256SAGNFI011, U4 DA9062-52AM1, U5 ATA6561-GBQW-N, U6 ATA6561-GBQW-N, U7 SM662GXC, Y1 32.768KHz, Y2 DSC6101JE3B-24MHz

Commit message: Update
Parts:
- removed U13: USBLC6-2SC6, Package_TO_SOT_SMD:SOT-23-6, symbol Power_Protection:USBLC6-2SC6
- added C140, C141, C226, C44: 100n, Capacitor_SMD:C_0402_1005Metric, symbol Device:C
- added D4, D6: CDSOD323-T05S, Diode_SMD:D_SOD-323, symbol Device:D_TVS_Filled
- added D5: CDSOD323-T03S, Diode_SMD:D_SOD-323, symbol Device:D_TVS_Filled
- added J5, J6: BK13H-30DP/2-0.35V05(895), HorizonPC:BK13H-30DP_2-0.35V05, symbol Connector_Generic_MountingPin:Conn_02x15_Row_Letter_Last_MountingPin
- added unit 18 of U1
- added U10, U9: ECMF02-2AMX6, Package_DFN_QFN:ST_UQFN-6L_1.5x1.7mm_P0.5mm, symbol Power_Protection:ECMF02-2AMX6
- added U8: PUSB3TB6AZ, HorizonPC:XSON7_PUSB3_NEX, symbol HorizonPC:PUSB3TB6AZ
- TP1: footprint TestPoint:TestPoint_Pad_D2.0mm -> TestPoint:TestPoint_Pad_D1.0mm
Connections:
- net +1.1V: now also U1.Y15 (PLL5_DVDD11), C140.1
- net +1.8V: now also U1.F17 (ADC_AVDD18), U1.Y11 (CSI_VDD18), U1.Y12 (CSI_VDD18), C141.1, C226.1, C44.1; no longer SW1.7
- net +3.3V: now also C160.1, R18.1, SW1.6, SW1.7; no longer C160.2
- net +5V: now also R2.1, R6.1, D6.1 (A1), J6.10a (Pin_10a), J6.10b (Pin_10b), J6.11a (Pin_11a), J6.11b (Pin_11b), J6.8b (Pin_8b), J6.9a (Pin_9a), J6.9b (Pin_9b)
- net +5V_EXT: no longer R2.1, R6.1
- net +5V_USB: now also D4.1 (A1), J6.5a (Pin_5a), J6.5b (Pin_5b), J6.6a (Pin_6a), J6.6b (Pin_6b), J6.7a (Pin_7a), J6.7b (Pin_7b), J6.8a (Pin_8a)
- net ADC_CH0: no longer U1.AE13 (ADC_CH0)
- net ADC_CH1: no longer U1.AD13 (ADC_CH1)
- net AUDIO_MCK: now also J5.4a (Pin_4a)
- net CAN0_STBY: now also U1.AC15 (P8_3); no longer U1.A17 (P18_1)
- net CAN1_STBY: now also U1.AC16 (P8_2); no longer U1.B17 (P18_2)
- net ETH_MDC: now also J4.9a (Pin_9a)
- net ETH_MDIO: now also J4.10a (Pin_10a)
- net ETH_RXC: now also J4.18a (Pin_18a)
- net ETH_RXD0: now also J4.16a (Pin_16a)
- net ETH_RXD1: now also J4.15a (Pin_15a)
- net ETH_RXD2: now also J4.13a (Pin_13a)
- net ETH_RXD3: now also J4.12a (Pin_12a)
- net ETH_RX_CTL: now also J4.20a (Pin_20a)
- net ETH_TXC: now also J4.18b (Pin_18b)
- net ETH_TXD0: now also J4.16b (Pin_16b)
- net ETH_TXD1: now also J4.15b (Pin_15b)
- net ETH_TXD2: now also J4.13b (Pin_13b)
- net ETH_TXD3: now also J4.12b (Pin_12b)
- net ETH_TX_CTL: now also J4.20b (Pin_20b)
- net GND: now also C160.2, J4.11a (Pin_11a), J4.11b (Pin_11b), J4.14a (Pin_14a), J4.14b (Pin_14b), J4.17a (Pin_17a), J4.17b (Pin_17b), J4.19a (Pin_19a), J4.19b (Pin_19b), J4.21a (Pin_21a), J4.21b (Pin_21b), J4.24a (Pin_24a), J4.27a (Pin_27a), J4.30a (Pin_30a), J4.33a (Pin_33a), J4.36a (Pin_36a), J4.38a (Pin_38a), J4.43a (Pin_43a), J4.43b (Pin_43b), J4.5a (Pin_5a), C140.2, C141.2, C226.2, C44.2, D4.2 (A2), D5.2 (A2), D6.2 (A2), J5.P1 (MountPin), J5.P2 (MountPin), J6.12a (Pin_12a), J6.12b (Pin_12b), J6.13a (Pin_13a), J6.13b (Pin_13b), J6.14a (Pin_14a), J6.14b (Pin_14b), J6.15a (Pin_15a), J6.15b (Pin_15b), J6.P2 (MountPin), U10.3 (GND), U8.1 (GND), U9.3 (GND); no longer C160.1
- net GPIO0_33: now also J4.37a (Pin_37a)
- net GPIO1_33: now also U1.B17 (P18_2), J5.7a (Pin_7a); no longer U1.AC16 (P8_2)
- net GPIO2_33: now also U1.A17 (P18_1), J5.11a (Pin_11a); no longer U1.AC15 (P8_3)
- net GPIO3_33: now also U1.F16 (P18_0), J5.4b (Pin_4b); no longer U1.A12 (P13_4)
- net GPIO4_33: now also J5.8a (Pin_8a)
- net GPIO5_33: now also U1.B12 (P13_3), J5.3b (Pin_3b); no longer U1.B2 (P24_0)
- net GPIO6_33: now also J5.6a (Pin_6a)
- net GPIO7_33: now also U1.A14 (P16_0), J5.10a (Pin_10a); no longer U1.B4 (P24_2)
- net GPIO8_33: now also U1.B14 (P16_1), J5.9a (Pin_9a); no longer U1.A3 (P24_3)
- net GPIO9_33: now also U1.A12 (P13_4), J5.2b (Pin_2b); no longer U1.B3 (P24_4)
- net IRQ0: now also J5.12a (Pin_12a)
- net IRQ3: now also J5.13a (Pin_13a)
- net IRQ4: now also J5.15b (Pin_15b)
- net JTAG_TCK: now also J4.4b (Pin_4b)
- net JTAG_TDI: now also J3.5 (Pin_5), J4.1b (Pin_1b); no longer J3.4 (Pin_4)
- net JTAG_TDO: now also J3.4 (Pin_4), J4.2b (Pin_2b); no longer J3.3 (Pin_3)
- net JTAG_TMS: now also J4.5b (Pin_5b)
- net JTAG_TRST#: now also J3.3 (Pin_3), J4.3b (Pin_3b); no longer J3.5 (Pin_5)
- net LDO2_EN: now also U1.B3 (P24_4); no longer U1.A14 (P16_0)
- net LDO3_EN: now also U1.A3 (P24_3); no longer U1.B14 (P16_1)
- net LDO4_EN: now also U1.B4 (P24_2); no longer U1.F16 (P18_0)
- net MAIN_RESET: now also J4.8a (Pin_8a)
- net MAIN_SCL: now also U1.B19 (RIIC0_SCL), J5.13b (Pin_13b); no longer U1.A19 (RIIC1_SCL)
- net MAIN_SDA: now also U1.B20 (RIIC0_SDA), J5.14b (Pin_14b); no longer U1.A20 (RIIC1_SDA)
- net MTU0_AB_DIS#: now also J5.3a (Pin_3a)
- net MTU0_CD_DIS#: now also J5.2a (Pin_2a)
- net MTU1_A: now also J4.10b (Pin_10b)
- net MTU1_AB_DIS#: now also J5.1a (Pin_1a)
- net MTU1_B: now also J4.9b (Pin_9b)
- net MTU1_C: now also J4.8b (Pin_8b)
- net MTU1_CD_DIS#: now also J5.1b (Pin_1b)
- net MTU1_D: now also J4.7b (Pin_7b)
- net NMI: now also J4.6b (Pin_6b)
- net PWR_ONKEY: now also J4.6a (Pin_6a)
- net PWR_SCL: now also U1.A19 (RIIC1_SCL); no longer U1.B19 (RIIC0_SCL)
- net PWR_SDA: now also U1.A20 (RIIC1_SDA); no longer U1.B20 (RIIC0_SDA)
- net PWR_WDT: now also U1.B2 (P24_0); no longer U1.B12 (P13_3)
- net PWR_WDT_ERR: now also J5.5a (Pin_5a)
- net SD1_CLK: now also U8.3 (CH2)
- net SD1_CMD: now also U8.6 (CH5)
- net SD1_D0: now also U8.5 (CH4)
- net SD1_D1: now also U8.4 (CH3)
- net SD1_D2: now also U8.7 (CH6)
- net SD1_D3: now also U8.2 (CH1)
- net SPI0_CLK: now also J5.8b (Pin_8b)
- net SPI0_MISO: now also J5.6b (Pin_6b)
- net SPI0_MOSI: now also J5.7b (Pin_7b)
- net SPI0_SSL: now also J5.5b (Pin_5b)
- net SPI1_CLK: now also J5.12b (Pin_12b)
- net SPI1_MISO: now also J5.10b (Pin_10b)
- net SPI1_MOSI: now also J5.11b (Pin_11b)
- net SPI1_SSL: now also J5.9b (Pin_9b)
- net SPI2_CLK: now also J4.41a (Pin_41a)
- net SPI2_MISO: now also J4.39a (Pin_39a)
- net SPI2_MOSI: now also J4.42a (Pin_42a)
- net SPI2_SSL: now also J4.40a (Pin_40a)
- net SYS_EN: now also J4.7a (Pin_7a)
- net USB+: now also U9.1 (D+_in)
- net USB-: now also U9.2 (D-_in)
- net USB_MAIN+: now also U10.2 (D-_in)
- net USB_MAIN-: now also U10.1 (D+_in)
- net VMAIN_RAW: now also J6.1a (Pin_1a), J6.1b (Pin_1b), J6.2a (Pin_2a), J6.2b (Pin_2b), J6.3a (Pin_3a), J6.3b (Pin_3b), J6.4a (Pin_4a), J6.4b (Pin_4b), J6.P1 (MountPin)
- net VSD1: now also D5.1 (A1); no longer R18.1, SW1.6
- net USB_ESD+: now reaches J4.1a (Pin_1a)
- net USB_ESD+: now also U9.6 (D+_out)
- net CSI_D3+: now reaches J4.22a (Pin_22a)
- net CSI_D3+: now also U1.AD9 (CSI_D3+)
- net CSI_D3-: now reaches J4.23a (Pin_23a)
- net CSI_D3-: now also U1.AE9 (CSI_D3-)
- net CSI_D1-: now reaches J4.25a (Pin_25a)
- net CSI_D1-: now also U1.AE10 (CSI_D1-)
- net CSI_D1+: now reaches J4.26a (Pin_26a)
- net CSI_D1+: now also U1.AD10 (CSI_D1+)
- net CSI_CLK-: now reaches J4.28a (Pin_28a)
- net CSI_CLK-: now also U1.AE11 (CSI_CLK-)
- net CSI_CLK+: now reaches J4.29a (Pin_29a)
- net CSI_CLK+: now also U1.AD11 (CSI_CLK+)
- net USB_ESD-: now reaches J4.2a (Pin_2a)
- net USB_ESD-: now also U9.5 (D-_out)
- net CSI_D0-: now reaches J4.31a (Pin_31a)
- net CSI_D0-: now also U1.AE12 (CSI_D0-)
- net CSI_D0+: now reaches J4.32a (Pin_32a)
- net CSI_D0+: now also U1.AD12 (CSI_D0+)
- net CSI_D2-: now reaches J4.34a (Pin_34a)
- net CSI_D2-: now also U1.AE13 (ADC_CH0)
- net CSI_D2+: now reaches J4.35a (Pin_35a)
- net CSI_D2+: now also U1.AD13 (ADC_CH1)
- net USB_MAIN_ESD-: now reaches J4.3a (Pin_3a)
- net USB_MAIN_ESD-: now also U10.6 (D+_out)
- net USB_MAIN_ESD+: now reaches J4.4a (Pin_4a)
- net USB_MAIN_ESD+: now also U10.5 (D-_out)
- new net: U1.B21 (NC), U1.F14 (NC)
- new net ADC_CH0_ARM: J5.14a (Pin_14a), U1.B18 (ADC_CH0)
- new net ADC_CH1_ARM: J5.15a (Pin_15a), U1.A18 (ADC_CH1)
Other:
- note added: "A18 / B18 only active with G2UL AD13 / AE13 only active with Rz/Five"
- note added: "MPU CSI"
- note added: "Main USB ESD"
- note added: "USB ESD"
- note added: "With G2UL: AE13 = CSI_D2- AD13 = CSI_D2+"
- note removed: "USB Connector"
- moved on the sheet: C160
